File: Fasanvej Rev1 Power.kicad_sch (KiCad schematic)
At the start: 50 parts

Commit message: Finished schematics. Pending validation.
Parts:
- added BT?: 18650, Battery:BatteryHolder_Keystone_1042_1x18650, symbol Device:Battery_Cell
- added C? (x2): 1u, Capacitor_SMD:C_0805_2012Metric_Pad1.18x1.45mm_HandSolder, symbol Device:C_Small
- added D?: D_Zener_Small, symbol Device:D_Zener_Small
- added L?: ???, symbol Device:L_Small
- added R?: 0R, Resistor_SMD:R_1210_3225Metric_Pad1.30x2.65mm_HandSolder, symbol Device:R_Small
- added R?: 5R, Resistor_SMD:R_1210_3225Metric_Pad1.30x2.65mm_HandSolder, symbol Device:R_Small
- added U?: AP5723WG-7, symbol RISRES Library:AP5723WG-7
Connections:
- net +BATT: now also C?.1, L?.1, U?.4 (EN), U?.6 (VIN)
- net GND: now also C?.2, C?.2, R?.1, R?.1, U?.2 (GND)
- net at BT?.2 (-), C?.2, Q?.3 (S)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: now also BT?.2 (-), R?.2
- net at BT?.1 (+), J?.2 (Pin_2), R?.1: now also BT?.1 (+)
- new net: D?.2 (A), L?.2, U?.1 (SW)
- new net LED_BACKLIGHT_A: R?.2, U?.3 (FB)
- new net LED_BACKLIGHT_K: C?.1, D?.1 (K), U?.5 (OVP)
Other:
- note added: "Backlight LED CC supply"
- note added: "Charge current 500 mA"
- note added: "Output current 20 mA"
- note added: "Protection override link"
- note removed: "Charge current = 500 mA"
- moved on the sheet: BT?, C?, D?, J?, L?, Q?, R?, SW?, U?
